File: Photon.kicad_sch (KiCad schematic)
At the start: 32 parts, among them P1 USB_C_6Pin, SW1 TS-1088-AR02016, U1 BQ24072RGTR, U2 ATtiny13A-S, U3 RT8059GJ5, U6 BCR421UW6-7, U7 BCR421UW6-7

Commit message: added new ic and started layout
Parts:
- removed P1: USB_C_6Pin, Connector_USB:USB_C_Receptacle_GCT_USB4125-xx-x-0190_6P_TopMnt_Horizontal, symbol Connector:USB_C_Plug_USB2.0
- removed TP4: LED1, TestPoint:TestPoint_Pad_D1.0mm, symbol Connector:TestPoint
- added C1, C3, C4: 4.7uF, Capacitor_SMD:C_0603_1608Metric, symbol Device:C
- added D1, D2: SZYY0603R1, LED_SMD:LED_0603_1608Metric, symbol Device:LED
- added J1: USB_C_Receptacle_USB2.0_14P, Connector_USB:USB_C_Receptacle_HRO_TYPE-C-31-M-17, symbol Connector:USB_C_Receptacle_USB2.0_14P
- added R11, R7: 1.18K, Resistor_SMD:R_0603_1608Metric, symbol Device:R
- added R13, R15, R4: 10K, Resistor_SMD:R_0603_1608Metric, symbol Device:R
- added R5: 0R, Resistor_SMD:R_0603_1608Metric, symbol Device:R
- added R6, R8: 1K, Resistor_SMD:R_0603_1608Metric, symbol Device:R
- added TP10: Vout, TestPoint:TestPoint_Pad_D1.0mm, symbol Connector:TestPoint
- added TP11: 3V6, TestPoint:TestPoint_Pad_D1.0mm, symbol Connector:TestPoint
- added TP12: LED1_EN, TestPoint:TestPoint_Pad_D1.0mm, symbol Connector:TestPoint
- added TP13: LED2_EN, TestPoint:TestPoint_Pad_D1.0mm, symbol Connector:TestPoint
- added TP8: BuckEN, TestPoint:TestPoint_Pad_D1.0mm, symbol Connector:TestPoint
- added TP9: BAT+, TestPoint:TestPoint_Pad_D1.0mm, symbol Connector:TestPoint
- D4, D5: If 20mA -> 20 to 50mA
- L1: value 2.2uH -> 4.7uH; footprint Photon:SMD 3.5x3mm Power Inductor -> Photon:SMD 3x3mm Power Inductor
- TP2: value LED2 -> VCC
- TP7: value VCC -> BTN
- U1: renamed from U2; footprint Package_SO:SOIC-8_5.3x5.3mm_P1.27mm -> Package_SO:SO-8_3.9x4.9mm_P1.27mm
- U3: renamed from U1; footprint (none) -> Photon:QFN-16_EP_3.8x3.8_Pitch0.5mm
- renumbered C4 to C5, C5 to C6, C1 to C7, R2 to R1, R5 to R10, R8 to R12, R9 to R14, R10 to R16, R1 to R2, R6 to R3, R4 to R9, TP8 to TP1, TP6 to TP3, TP5 to TP4, TP3 to TP5, TP1 to TP6, U3 to U2, U6 to U4, U7 to U5
Connections:
- net +BATT is gone; now on net BAT: BT1.1 (+)
- net -BATT is gone; now on net GND: BT1.2 (-)
- net 3V6: now also C1.2, TP11.1; no longer TP7.1
- net CC1: now also J1.A5 (CC1)
- net CC2: now also J1.B5 (CC2)
- net GND: now also U3.15 (TD), U3.4 (CE), U3.6 (EN1), U3.8 (VSS), C1.1, C3.1, C4.1, J1.A1 (GND), J1.A12 (GND), J1.B1 (GND), J1.B12 (GND), J1.S1 (SHIELD), R11.2, R13.2, R15.2, R4.1, R5.2, R7.2
- net LED1_EN: now also R13.1, TP12.1
- net LED2_EN: now also R15.1, TP13.1; no longer TP2.1
- net MISO_BTN: now also TP7.1
- net VCC: now also TP2.1, U3.13 (IN), C4.2, J1.A4 (VBUS), J1.A9 (VBUS), J1.B4 (VBUS), J1.B9 (VBUS)
- net VOUT: now also U3.5 (EN2), R6.1, R8.1, TP10.1, TP8.1
- net TS: now reaches U3.1 (TS)
- net TS: now also R4.2
- net ILIM: now reaches U3.12 (ILIM)
- net ILIM: now also R7.1
- net TMR: now reaches U3.14 (TMR)
- net TMR: now also R5.1
- net ISET: now reaches U3.16 (ISET)
- net ISET: now also R11.1
- net BAT: now reaches U3.2 (BAT)
- net BAT: now also U3.3 (BAT), C3.2, TP9.1
- net PGOOD: now reaches U3.7 (PGOOD)
- net PGOOD: now also D1.1 (K)
- net CHG: now reaches U3.9 (CHG)
- net CHG: now also D2.1 (K)
- new net G_A: D1.2 (A), R6.2
- new net R_A: D2.2 (A), R8.2
- no-connect marks 0 -> 4
Other:
- note added: "18650 Battery Vout=3.7-4.2V"
- note added: "Vo = 0.6 * (1+R1/R2) R2 = 60K to 300K"
- note removed: "18650 Battery Cell holder Vout=3.7-4.2V"
- note removed: "Probe Points"
- moved on the sheet: BT1, C2, C5, C6, C7, D3, D4, D5, L1, R1, R10, R12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

Commit message: Added TP4056 back
Parts:
- removed TP10: Vout, TestPoint:TestPoint_Pad_D1.0mm, symbol Connector:TestPoint
- added C10, C9: 10uF, Capacitor_SMD:C_0603_1608Metric, symbol Device:C
- added C8: 0.1uF, Capacitor_SMD:C_0603_1608Metric, symbol Device:C
- added D6, D7: SZYY0603R1, LED_SMD:LED_0603_1608Metric, symbol Device:LED
- added R17: 100R, Resistor_SMD:R_0603_1608Metric, symbol Device:R
- added R18, R20, R21: 1K, Resistor_SMD:R_0603_1608Metric, symbol Device:R
- added R19: 2K, Resistor_SMD:R_0603_1608Metric, symbol Device:R
- added U6: DW01A, Package_TO_SOT_SMD:SOT-23-6, symbol Photon:DW01A
- added U7: FS8205A, Package_TO_SOT_SMD:SOT-23-6, symbol Photon:FS8205A
- added U8: TP4056, Package_SO:SOIC-8-1EP_3.9x4.9mm_P1.27mm_EP2.29x3mm, symbol Photon:TP4056
- TP2: value VCC -> 5V
Connections:
- net GND: now also C10.1, C9.1, R18.1, R19.2, U7.3 (S2), U8.3 (VSS); no longer BT1.2 (-)
- net VCC: no longer C4.2, J1.A4 (VBUS), J1.A9 (VBUS), J1.B4 (VBUS), J1.B9 (VBUS), TP2.1, U3.13 (IN)
- net VOUT: no longer C2.2, TP8.1, U2.1 (EN), U2.4 (Vin)
- net BAT renamed PACK+
- net PACK+: now also C2.2, TP8.1, U2.1 (EN), U2.4 (Vin), C9.2, R17.1, U8.5 (VBAT)
- new net: D6.2 (A), R21.2
- new net: D7.1 (K), U8.6 (STAT2)
- new net: D7.2 (A), R20.2
- new net: R19.1, U8.2 (ISET)
- new net: D6.1 (K), U8.7 (STAT1)
- new net: R18.2, U6.2 (VM)
- new net: BT1.2 (-), C8.1, U6.6 (GND), U7.1 (S1)
- new net: U6.3 (OC), U7.4 (G2)
- new net: U6.1 (OD), U7.6 (G1)
- new net: C8.2, R17.2, U6.5 (VCC)
- new net 5V: C10.2, C4.2, J1.A4 (VBUS), J1.A9 (VBUS), J1.B4 (VBUS), J1.B9 (VBUS), R20.1, R21.1, TP2.1, U3.13 (IN), U8.4 (VIN), U8.8 (EN)
- no-connect marks 4 -> 7
Other:
- note added: "ATTINY"
- note added: "Voltage Regulator 3V6"
- note removed: "Buck"
- note removed: "Controller"
- moved on the sheet: BT1, C1, C2, C3, C4, C5, C6, C7, D1, D2, D3, D4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
