File: PCB/Photon.kicad_sch (KiCad schematic)
At the start: 44 parts, among them J1 USB_C_Receptacle_USB2.0_14P, J2 Conn_01x05_Socket, Q1 IRLML6402, Q2 IRLML6402, SW1 TS-1088-AR02016, U1 PY32F002AL15S6TU, U2 TP4056, U3 RT8059GJ5, U4 BCR421UW6-7, U5 DW01A, U6 FS8205A, U7 BCR421UW6-7

Commit message: Squashed commit of the following:
commit 040f56c92c5fbfa60c6357d084ca9e817f85bd74
Author: AirMatress <134566567+Kay-Jack@users.noreply.github.com>
Date:   Sun Feb 15 22:31:25 2026 -0500

    changed folder structure and added new photos

commit a5de8e0470fd1fbaa1884b4c13b8efd9701bd3f9
Author: AirMatress <134566567+Kay-Jack@users.noreply.github.com>
Date:   Sun Feb 15 22:04:27 2026 -0500

    added zip

commit 86241a126469fe2acf0b48b8ae5ce0ab9d585c9c
Author: AirMatress <134566567+Kay-Jack@users.noreply.github.com>
Date:   Sun Feb 15 21:56:49 2026 -0500

    added gerbers

commit 35698b9b92e03ab22e12582723e18a858d02b47b
Author: AirMatress <134566567+Kay-Jack@users.noreply.github.com>
Date:   Sun Feb 15 21:54:39 2026 -0500

    switch to smt32 mcu and cleaned up pcb

commit b81d1645440da80b902de656f60b2bd3905a4b55
Author: AirMatress <134566567+Kay-Jack@users.noreply.github.com>
Date:   Sun Jan 18 22:33:01 2026 -0500

    updated debug header and changed resistors for UVLO

    Applied teardrop to all vias. some were missing. Thickened trace from neg battery terminal. Updated gerbers

commit b8795243000142daf8d6161322fd58468c0a1805
Author: AirMatress <134566567+Kay-Jack@users.noreply.github.com>
Date:   Mon Jan 5 22:00:06 2026 -0500

    Rotated PCB

commit 89b92c6a3bacb1a8dd3ef43ffdd3007030cc7a51
Author: AirMatress <134566567+Kay-Jack@users.noreply.github.com>
Date:   Mon Jan 5 21:30:51 2026 -0500

    updated photos and added path for step of tp4056

commit 6c3586d8c21dee7771f43999eac4c35423b5389e
Author: AirMatress <134566567+AirMatress@users.noreply.github.com>
Date:   Thu Jan 1 13:02:22 2026 -0500

    added UVLO for the buck
Parts:
- removed TP10: LED1_EN, TestPoint:TestPoint_THTPad_D1.0mm_Drill0.5mm, symbol Connector:TestPoint
- removed TP11: LED2_EN, TestPoint:TestPoint_THTPad_D1.0mm_Drill0.5mm, symbol Connector:TestPoint
- removed TP6: 5V, TestPoint:TestPoint_THTPad_D1.0mm_Drill0.5mm, symbol Connector:TestPoint
- removed U1: PY32F002AL15S6TU, Package_SO:SOP-8_3.9x4.9mm_P1.27mm, symbol Photon:PY32F002AL15S6TU
- added C2: 100nF, Capacitor_SMD:C_0603_1608Metric, symbol Device:C
- added R5: 12K, Resistor_SMD:R_0603_1608Metric, symbol Device:R
- added U1: STM32G030F6P6TR, Package_SO:TSSOP-20_4.4x6.5mm_P0.65mm, symbol MCU_ST_STM32G0:STM32G030F6Px
- C1: value 100nF -> 4.7uF; footprint Capacitor_SMD:C_0603_1608Metric -> Capacitor_SMD:C_0805_2012Metric
- J1: value USB_C_Receptacle_USB2.0_14P -> USB_C_Receptacle_USB2.0_6P
- R6: value 100K -> 10K
- renumbered C2 to C4, C6 to C5, C4 to C6, C5 to C7, C7 to C8, R9 to R10, R14 to R11, R13 to R12, R17 to R13, R19 to R14, R16 to R15, R7 to R3, R10 to R4, R4 to R7, R5 to R8, R8 to R9, U5 to U4, U6 to U5, U4 to U6
Connections:
- net +3V3: now also J2.1 (Pin_1), C2.1, U1.4 (VDD); no longer J2.5 (Pin_5)
- net GND: now also J2.5 (Pin_5), C2.2, U1.5 (VSS); no longer J2.1 (Pin_1)
- net LED1_EN: now also U1.13 (PA6)
- net LED2_EN: now also U1.14 (PA7)
- net NRST: now also U1.6 (NRST)
- net VBAT_SYS: now also R5.1; no longer R6.1, U3.1 (EN)
- net BTN renamed BUTN
- net BUTN: now also U1.12 (PA5)
- net SWC renamed SWCLK
- net SWCLK: now also U1.19 (PA14/PA15)
- net SWD renamed SWDIO
- net SWDIO: now also U1.18 (PA13)
- new net UVLO: R5.2, R6.1, U3.1 (EN)
- no-connect marks 7 -> 19
Other:
- note added: "UVLO 3.3V"
- moved on the sheet: J2, R6, SW1
